File: PCB/Blitzypad.kicad_pcb (KiCad board)
At the start: 2 copper layers, 97.6 x 62.4 mm, 10 parts, among them SW1 SW_Push, SW2 SW_Push, SW3 SW_Push, SW4 SW_Push, SW5 RotaryEncoder_Switch, SW6 SW_Push, U1 XIAO-RP2040-DIP, U2 OLED_0.91_128x32

Commit message: Apply fixes according to feedback
Connections:
- U1 pad 14: unconnected-(U1-VBUS-Pad14) -> +5V
Routing:
- net +5V: track 10.3 -> 19.9 mm, vias 0 -> 1
Changed lines of the file:
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@@
 	(net 10 "Net-(U1-GPIO27{slash}ADC1{slash}A1)")
 	(net 11 "Net-(U1-GPIO28{slash}ADC2{slash}A2)")
-	(net 12 "unconnected-(U1-VBUS-Pad14)")
-	(net 13 "Net-(U1-GPIO26{slash}ADC0{slash}A0)")
-	(net 14 "+5V")
-	(net 15 "Net-(D1-DOUT)")
-	(net 16 "unconnected-(D2-DOUT-Pad2)")
-	(net 17 "Net-(U1-GPIO29{slash}ADC3{slash}A3)")
+	(net 12 "Net-(U1-GPIO26{slash}ADC0{slash}A0)")
+	(net 13 "+5V")
+	(net 14 "Net-(D1-DOUT)")
+	(net 15 "unconnected-(D2-DOUT-Pad2)")
+	(net 16 "Net-(U1-GPIO29{slash}ADC3{slash}A3)")
 	(footprint "hkcl:OLED_0.91_128x32"
 		(layer "F.Cu")
@@
 			(layers "*.Cu" "*.Mask")
 			(remove_unused_layers no)
-			(net 13 "Net-(U1-GPIO26{slash}ADC0{slash}A0)")
+			(net 12 "Net-(U1-GPIO26{slash}ADC0{slash}A0)")
 			(pinfunction "B")
 			(pintype "passive")
@@
 			(layers "B.Cu" "B.Mask" "B.Paste")
 			(roundrect_rratio 0.1)
-			(net 14 "+5V")
+			(net 13 "+5V")
 			(pinfunction "VDD")
 			(pintype "power_in")
@@
 			(layers "B.Cu" "B.Mask" "B.Paste")
 			(roundrect_rratio 0.1)
-			(net 15 "Net-(D1-DOUT)")
+			(net 14 "Net-(D1-DOUT)")
 			(pinfunction "DOUT")
 			(pintype "output")
@@
 			(layers "*.Cu" "*.Mask")
 			(remove_unused_layers no)
-			(net 17 "Net-(U1-GPIO29{slash}ADC3{slash}A3)")
+			(net 16 "Net-(U1-GPIO29{slash}ADC3{slash}A3)")
 			(pinfunction "2")
 			(pintype "passive")
@@
 			(layers "B.Cu" "B.Mask" "B.Paste")
 			(roundrect_rratio 0.1)
-			(net 14 "+5V")
+			(net 13 "+5V")
 			(pinfunction "VDD")
 			(pintype "power_in")
@@
 			(layers "B.Cu" "B.Mask" "B.Paste")
 			(roundrect_rratio 0.1)
-			(net 16 "unconnected-(D2-DOUT-Pad2)")
+			(net 15 "unconnected-(D2-DOUT-Pad2)")
 			(pinfunction "DOUT")
 			(pintype "output")
@@
 			(layers "B.Cu" "B.Mask" "B.Paste")
 			(roundrect_rratio 0.1)
-			(net 15 "Net-(D1-DOUT)")
+			(net 14 "Net-(D1-DOUT)")
 			(pinfunction "DIN")
 			(pintype "input")
@@
 			(layers "F.Cu" "F.Mask")
 			(roundrect_rratio 0.1)
-			(net 13 "Net-(U1-GPIO26{slash}ADC0{slash}A0)")
+			(net 12 "Net-(U1-GPIO26{slash}ADC0{slash}A0)")
 			(pinfunction "GPIO26/ADC0/A0")
 			(pintype "passive")
@@
 			(layers "*.Cu" "*.Mask")
 			(remove_unused_layers no)
-			(net 13 "Net-(U1-GPIO26{slash}ADC0{slash}A0)")
+			(net 12 "Net-(U1-GPIO26{slash}ADC0{slash}A0)")
 			(pinfunction "GPIO26/ADC0/A0")
 			(pintype "passive")
@@
 			(layers "F.Cu" "F.Mask")
 			(roundrect_rratio 0.1)
-			(net 17 "Net-(U1-GPIO29{slash}ADC3{slash}A3)")
+			(net 16 "Net-(U1-GPIO29{slash}ADC3{slash}A3)")
 			(pinfunction "GPIO29/ADC3/A3")
 			(pintype "passive")
@@
 			(layers "*.Cu" "*.Mask")
 			(remove_unused_layers no)
-			(net 17 "Net-(U1-GPIO29{slash}ADC3{slash}A3)")
+			(net 16 "Net-(U1-GPIO29{slash}ADC3{slash}A3)")
 			(pinfunction "GPIO29/ADC3/A3")
 			(pintype "passive")
@@
 			(layers "*.Cu" "*.Mask")
 			(remove_unused_layers no)
-			(net 12 "unconnected-(U1-VBUS-Pad14)")
+			(net 13 "+5V")
 			(pinfunction "VBUS")
 			(pintype "passive")
@@
 			(layers "F.Cu" "F.Mask")
 			(roundrect_rratio 0.1)
-			(net 12 "unconnected-(U1-VBUS-Pad14)")
+			(net 13 "+5V")
 			(pinfunction "VBUS")
 			(pintype "passive")
@@
 		(width 0.2)
 		(layer "F.Cu")
-		(net 13)
+		(net 12)
 	)
 	(segment
@@
 		(width 0.2)
 		(layer "F.Cu")
-		(net 13)
+		(net 12)
 	)
 	(segment
@@
 		(width 0.2)
 		(layer "F.Cu")
-		(net 13)
+		(net 12)
 	)
 	(segment
@@
 		(width 0.2)
 		(layer "F.Cu")
-		(net 13)
+		(net 12)
 	)
 	(segment
@@
 		(width 0.2)
 		(layer "F.Cu")
-		(net 13)
+		(net 12)
 	)
 	(segment
@@
 		(width 0.2)
 		(layer "F.Cu")
-		(net 13)
+		(net 12)
 	)
 	(segment
@@
 		(width 0.2)
 		(layer "F.Cu")
-		(net 13)
+		(net 12)
 	)
 	(segment
@@
 		(width 0.2)
 		(layer "F.Cu")
+		(net 12)
+	)
+	(segment
+		(start 199 78.54237)
+		(end 196.65763 76.2)
+		(width 0.2)
+		(layer "F.Cu")
+		(net 13)
+	)
+	(segment
+		(start 196.65763 76.2)
+		(end 195.58 76.2)
+		(width 0.2)
+		(layer "F.Cu")
+		(net 13)
+	)
+	(segment
+		(start 199 80)
+		(end 199 78.54237)
+		(width 0.2)
+		(layer "F.Cu")
+		(net 13)
+	)
+	(via
+		(at 199 80)
+		(size 0.6)
+		(drill 0.3)
+		(layers "F.Cu" "B.Cu")
 		(net 13)
 	)
@@
 		(width 0.2)
 		(layer "B.Cu")
-		(net 14)
+		(net 13)
 	)
 	(segment
@@
 		(width 0.2)
 		(layer "B.Cu")
-		(net 14)
+		(net 13)
 	)
 	(segment
@@
 		(width 0.2)
 		(layer "B.Cu")
-		(net 14)
+		(net 13)
+	)
+	(segment
+		(start 202.267671 80.732329)
+		(end 201.535342 80)
+		(width 0.2)
+		(layer "B.Cu")
+		(net 13)
+	)
+	(segment
+		(start 202.40625 80.870909)
+		(end 202.267671 80.732329)
+		(width 0.2)
+		(layer "B.Cu")
+		(net 13)
 	)
 	(segment
@@
 		(width 0.2)
 		(layer "B.Cu")
-		(net 14)
+		(net 13)
+	)
+	(segment
+		(start 201.535342 80)
+		(end 199 80)
+		(width 0.2)
+		(layer "B.Cu")
+		(net 13)
 	)
 	(segment
@@
 		(width 0.2)
 		(layer "B.Cu")
-		(net 15)
+		(net 14)
 	)
 	(segment
@@
 		(width 0.2)
 		(layer "B.Cu")
-		(net 15)
+		(net 14)
 	)
 	(segment
@@
 		(width 0.2)
 		(layer "B.Cu")
-		(net 15)
+		(net 14)
 	)
 	(segment
@@
 		(width 0.2)
 		(layer "B.Cu")
-		(net 15)
+		(net 14)
 	)
 	(segment
@@
 		(width 0.2)
 		(layer "B.Cu")
-		(net 15)
+		(net 14)
 	)
 	(segment
@@
 		(width 0.2)
 		(layer "B.Cu")
-		(net 15)
+		(net 14)
 	)
 	(segment
@@
 		(width 0.2)
 		(layer "F.Cu")
-		(net 17)
+		(net 16)
 	)
 	(segment
@@
 		(width 0.2)
 		(layer "F.Cu")
-		(net 17)
+		(net 16)
 	)
 	(segment
@@
 		(width 0.2)
 		(layer "F.Cu")
-		(net 17)
+		(net 16)
 	)
 	(segment
@@
 		(width 0.2)
 		(layer "F.Cu")
-		(net 17)
+		(net 16)
 	)
 	(segment
@@
 		(width 0.2)
 		(layer "F.Cu")
-		(net 17)
+		(net 16)
 	)
 	(group ""

Commit message: small pcb changes to make it look nicer
Routing:
- net Net-(D1-DOUT): track 16.1 -> 9.91 mm
- net Net-(U1-GPIO4/MISO): track 48.8 -> 53.9 mm, vias 1 -> 0
- net GND: track 225.5 -> 230.6 mm
- net Net-(D1-DIN): track 65.1 -> 60.9 mm
- net Net-(U1-GPIO2/SCK): track 21.7 -> 22.5 mm
- net +5V: track 19.9 -> 20.1 mm, vias 1 -> 0
